File: PowerCastel.brd (EAGLE design)
At the start: 31.8 x 19.1 mm, 22 parts, among them U1 TPS61090RSAR, U2 MCP73871

Commit message: Fixed ground planes and added power planes
Ground plane connection to components on left side of board has been widened. Added power planes as specified by TPS61090 datasheet.
Routing:
- net GND: track 18.3 -> 9.67 mm, vias 4 -> 10
- net 5.0V: track 21.6 -> 13.6 mm
- net N$1: track 5.33 -> 2.41 mm
- net ENABLE: track 26.2 -> 25.0 mm
- net VBUS: track 25.1 -> 24.3 mm
- added copper zone on layer 1, net 5.0V
- added copper zone on layer 1, net N$1
Other:
- board size 31.8 x 19.1 mm -> 27.9 x 17.1 mm
Changed lines of the file:
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@@
 <board>
 <plain>
-<wire x1="0" y1="0" x2="31.75" y2="0" width="0" layer="20"/>
-<wire x1="31.75" y1="0" x2="31.75" y2="19.05" width="0" layer="20"/>
-<wire x1="31.75" y1="19.05" x2="0" y2="19.05" width="0" layer="20"/>
-<wire x1="0" y1="19.05" x2="0" y2="0" width="0" layer="20"/>
+<wire x1="1.27" y1="1.905" x2="29.21" y2="1.905" width="0" layer="20"/>
+<wire x1="29.21" y1="1.905" x2="29.21" y2="19.05" width="0" layer="20"/>
+<wire x1="29.21" y1="19.05" x2="1.27" y2="19.05" width="0" layer="20"/>
+<wire x1="1.27" y1="19.05" x2="1.27" y2="1.905" width="0" layer="20"/>
 <text x="14.605" y="15.24" size="1.27" layer="22" rot="MR90" align="center-right">BAT</text>
 <text x="17.145" y="15.24" size="1.27" layer="22" rot="MR90" align="center-right">GND</text>
@@
 <contactref element="R17" pad="1"/>
 <contactref element="J2" pad="1"/>
-<polygon width="0.3048" layer="1">
+<polygon width="0.3048" layer="1" thermals="no" rank="2">
 <vertex x="3.81" y="16.51"/>
 <vertex x="27.305" y="16.51"/>
@@
 <vertex x="3.175" y="16.51"/>
 </polygon>
-<polygon width="0.3048" layer="16">
+<polygon width="0.3048" layer="16" thermals="no" rank="2">
 <vertex x="3.175" y="16.51"/>
 <vertex x="27.305" y="16.51"/>
@@
 <wire x1="10.398" y1="9.287" x2="9.398" y2="10.287" width="0.3048" layer="1"/>
 <wire x1="11.363" y1="9.414" x2="10.398" y2="9.414" width="0.3048" layer="1"/>
-<wire x1="18.09" y1="11.498" x2="18.09" y2="9.723" width="0.3048" layer="1"/>
 <wire x1="18.09" y1="9.723" x2="18.415" y2="9.398" width="0.3048" layer="1"/>
-<wire x1="18.74" y1="11.498" x2="18.74" y2="9.723" width="0.3048" layer="1"/>
 <wire x1="18.74" y1="9.723" x2="18.415" y2="9.398" width="0.3048" layer="1"/>
-<wire x1="19.39" y1="11.498" x2="19.39" y2="10.373" width="0.3048" layer="1"/>
 <wire x1="19.39" y1="10.373" x2="19.315" y2="10.298" width="0.3048" layer="1"/>
-<wire x1="18.74" y1="11.498" x2="18.74" y2="12.695" width="0.3048" layer="1"/>
 <wire x1="18.74" y1="12.695" x2="18.481" y2="12.954" width="0.3048" layer="1"/>
-<wire x1="18.09" y1="11.498" x2="18.09" y2="12.563" width="0.3048" layer="1"/>
 <wire x1="18.09" y1="12.563" x2="18.481" y2="12.954" width="0.3048" layer="1"/>
-<wire x1="19.39" y1="11.498" x2="19.39" y2="12.36" width="0.3048" layer="1"/>
 <wire x1="18.796" y1="12.954" x2="18.481" y2="12.954" width="0.3048" layer="1"/>
-<wire x1="19.39" y1="12.36" x2="18.796" y2="12.954" width="0.3048" layer="1"/>
 <wire x1="18.415" y1="9.398" x2="17.44" y2="8.423" width="0.3048" layer="1"/>
 <wire x1="17.44" y1="8.423" x2="17.44" y2="7.298" width="0.3048" layer="1"/>
@@
 <via x="10.795" y="15.24" extent="1-16" drill="0.35"/>
 <via x="6.35" y="14.732" extent="1-16" drill="0.35"/>
+<via x="10.16" y="5.969" extent="1-16" drill="0.35"/>
+<via x="25.1714" y="5.8166" extent="1-16" drill="0.35"/>
+<via x="26.3398" y="6.223" extent="1-16" drill="0.35"/>
+<via x="26.4414" y="7.5438" extent="1-16" drill="0.35"/>
+<via x="26.416" y="8.763" extent="1-16" drill="0.35"/>
+<wire x1="10.398" y1="8.449" x2="10.16" y2="5.969" width="0" layer="19" extent="1-1"/>
+<via x="5.2832" y="5.715" extent="1-16" drill="0.35"/>
 </signal>
 <signal name="N$1">
@@
 <contactref element="U1" pad="4"/>
 <contactref element="L1" pad="P$2"/>
-<wire x1="20.515" y1="10.373" x2="21.844" y2="10.373" width="0.3048" layer="1"/>
 <wire x1="21.844" y1="10.373" x2="23.403" y2="10.373" width="0.3048" layer="1"/>
 <wire x1="23.403" y1="10.373" x2="24.003" y2="10.973" width="0.3048" layer="1"/>
-<wire x1="20.515" y1="9.723" x2="21.194" y2="9.723" width="0.3048" layer="1"/>
-<wire x1="21.194" y1="9.723" x2="21.844" y2="10.373" width="0.3048" layer="1"/>
+<polygon width="0.1016" layer="1" thermals="no">
+<vertex x="20.0406" y="10.4902"/>
+<vertex x="21.0058" y="10.4902"/>
+<vertex x="21.5392" y="11.0236"/>
+<vertex x="21.5646" y="11.049"/>
+<vertex x="21.5646" y="11.3284"/>
+<vertex x="21.5646" y="11.9126"/>
+<vertex x="26.4414" y="11.9126"/>
+<vertex x="26.4414" y="10.033"/>
+<vertex x="21.3614" y="10.033"/>
+<vertex x="20.9296" y="9.6012"/>
+<vertex x="20.0406" y="9.6012"/>
+</polygon>
 </signal>
 <signal name="N$3">
@@
 <contactref element="C6" pad="1"/>
 <contactref element="J2" pad="2"/>
-<wire x1="20.515" y1="8.423" x2="21.927" y2="8.423" width="0.3048" layer="1"/>
 <wire x1="21.927" y1="8.423" x2="22.222" y2="8.128" width="0.3048" layer="1"/>
-<wire x1="19.39" y1="7.298" x2="18.74" y2="7.298" width="0.3048" layer="1"/>
 <wire x1="22.222" y1="7.49" x2="22.222" y2="7.874" width="0.3048" layer="1"/>
 <wire x1="22.222" y1="7.874" x2="22.222" y2="8.128" width="0.3048" layer="1"/>
 <wire x1="22.03" y1="7.298" x2="22.222" y2="7.49" width="0.3048" layer="1"/>
-<wire x1="22.037" y1="5.842" x2="22.037" y2="7.689" width="0.3048" layer="1"/>
 <wire x1="22.037" y1="7.689" x2="22.222" y2="7.874" width="0.3048" layer="1"/>
-<wire x1="19.39" y1="7.298" x2="20.193" y2="7.298" width="0.3048" layer="1"/>
-<wire x1="20.193" y1="7.298" x2="22.03" y2="7.298" width="0.3048" layer="1"/>
-<wire x1="20.254" y1="5.842" x2="20.254" y2="7.237" width="0.3048" layer="1"/>
-<wire x1="20.254" y1="7.237" x2="20.193" y2="7.298" width="0.3048" layer="1"/>
 <via x="23.622" y="8.128" extent="1-16" drill="0.35"/>
 <wire x1="22.225" y1="16.51" x2="25.6032" y2="13.1318" width="0.8128" layer="16"/>
@@
 <wire x1="23.622" y1="9.40820625" x2="23.622" y2="8.128" width="0.8128" layer="16"/>
 <wire x1="23.622" y1="8.128" x2="22.222" y2="8.128" width="0.8128" layer="1"/>
+<polygon width="0.1016" layer="1" thermals="no">
+<vertex x="18.6182" y="7.7724"/>
+<vertex x="20.0406" y="7.7724"/>
+<vertex x="20.0406" y="9.1948"/>
+<vertex x="21.209" y="9.1948"/>
+<vertex x="21.4376" y="9.4234"/>
+<vertex x="22.9616" y="9.4234"/>
+<vertex x="22.9616" y="6.8326"/>
+<vertex x="22.6314" y="6.8326"/>
+<vertex x="22.6314" y="5.1562"/>
+<vertex x="19.6596" y="5.1562"/>
+<vertex x="19.6596" y="6.3246"/>
+<vertex x="19.6596" y="6.8326"/>
+<vertex x="18.6436" y="6.8326"/>
+<vertex x="18.6182" y="6.8326"/>
+</polygon>
 </signal>
 <signal name="VBAT">
@@
 <wire x1="4.3332" y1="14.859" x2="4.3332" y2="14.732" width="0.3048" layer="1"/>
 <wire x1="4.3332" y1="14.732" x2="4.3332" y2="13.335" width="0.3048" layer="1"/>
-<via x="5.207" y="14.605" extent="1-16" drill="0.35"/>
-<wire x1="5.207" y1="14.605" x2="4.3332" y2="14.605" width="0.3048" layer="1"/>
+<via x="5.2832" y="14.5288" extent="1-16" drill="0.35"/>
+<wire x1="5.2832" y1="14.5288" x2="4.3332" y2="14.5288" width="0.3048" layer="1"/>
 <via x="13.462" y="10.16" extent="1-16" drill="0.35"/>
-<wire x1="5.207" y1="14.605" x2="5.207" y2="8.128" width="0.3048" layer="16"/>
-<wire x1="7.493" y1="5.842" x2="10.16" y2="5.842" width="0.3048" layer="16"/>
-<wire x1="10.16" y1="5.842" x2="13.462" y2="9.144" width="0.3048" layer="16"/>
-<wire x1="13.462" y1="9.144" x2="13.462" y2="10.16" width="0.3048" layer="16"/>
-<wire x1="5.207" y1="8.128" x2="7.493" y2="5.842" width="0.3048" layer="16"/>
+<wire x1="5.2832" y1="14.5288" x2="5.2832" y2="8.0518" width="0.3048" layer="16"/>
+<wire x1="6.6294" y1="6.7056" x2="10.1092" y2="6.7056" width="0.3048" layer="16"/>
+<wire x1="10.1092" y1="6.7056" x2="13.462" y2="10.0584" width="0.3048" layer="16"/>
+<wire x1="13.462" y1="10.0584" x2="13.462" y2="10.16" width="0.3048" layer="16"/>
+<wire x1="5.2832" y1="8.0518" x2="6.6294" y2="6.7056" width="0.3048" layer="16"/>
 <wire x1="13.462" y1="10.16" x2="13.716" y2="9.906" width="0.3048" layer="1"/>
 <wire x1="13.716" y1="9.906" x2="13.716" y2="9.271" width="0.3048" layer="1"/>
@@
 <wire x1="14.097" y1="8.89" x2="15.52405" y2="8.89" width="0.3048" layer="1"/>
 <wire x1="15.52405" y1="8.89" x2="15.70705" y2="9.073" width="0.3048" layer="1"/>
-<wire x1="4.3332" y1="14.859" x2="4.3332" y2="14.605" width="0.3048" layer="1"/>
+<wire x1="4.3332" y1="14.859" x2="4.3332" y2="14.5288" width="0.3048" layer="1"/>
 </signal>
 <signal name="N$5">
@@
 <wire x1="9.398" y1="13.335" x2="9.898" y2="12.835" width="0.254" layer="1"/>
 <wire x1="9.898" y1="12.835" x2="9.898" y2="12.379" width="0.254" layer="1"/>
-<wire x1="6.985" y1="16.51" x2="6.985" y2="15.748" width="0.8128" layer="16"/>
-<wire x1="6.985" y1="15.748" x2="9.398" y2="13.335" width="0.8128" layer="16"/>
 <wire x1="7.433" y1="9.914" x2="6.292" y2="9.914" width="0.254" layer="1"/>
 <wire x1="6.292" y1="9.914" x2="6.096" y2="9.718" width="0.254" layer="1"/>
@@
 <via x="6.096" y="8.5344" extent="1-16" drill="0.35"/>
 <wire x1="6.096" y1="12.7" x2="6.731" y2="13.335" width="0.8128" layer="16"/>
-<wire x1="6.096" y1="8.5344" x2="8.0264" y2="6.604" width="0.8128" layer="16"/>
-<wire x1="8.0264" y1="6.604" x2="9.144" y2="6.604" width="0.8128" layer="16"/>
-<via x="9.144" y="6.604" extent="1-16" drill="0.35"/>
+<wire x1="6.096" y1="8.5344" x2="7.0866" y2="7.5438" width="0.8128" layer="16"/>
+<wire x1="7.0866" y1="7.5438" x2="9.906" y2="7.5438" width="0.8128" layer="16"/>
+<via x="9.906" y="7.5438" extent="1-16" drill="0.35"/>
 <wire x1="6.096" y1="8.5344" x2="6.096" y2="12.7" width="0.8128" layer="16"/>
 <wire x1="6.731" y1="13.335" x2="9.398" y2="13.335" width="0.8128" layer="16"/>
-<wire x1="9.898" y1="8.449" x2="9.898" y2="7.358" width="0.2032" layer="1"/>
-<wire x1="9.898" y1="7.358" x2="9.144" y2="6.604" width="0.2032" layer="1"/>
+<wire x1="9.898" y1="8.449" x2="9.898" y2="7.5518" width="0.2032" layer="1"/>
+<wire x1="9.906" y1="7.5438" x2="9.898" y2="7.5518" width="0.2032" layer="1"/>
+<wire x1="6.985" y1="16.51" x2="9.398" y2="14.097" width="0.8128" layer="1"/>
+<wire x1="9.398" y1="14.097" x2="9.398" y2="13.335" width="0.8128" layer="1"/>
 </signal>
 <signal name="VLIPO">

Commit message: Fixed ground via
Routing:
- net GND: track 9.67 -> 4.07 mm, vias 10 -> 11
- net N$1: track 2.41 -> 0.00 mm
- net 5.0V: track 13.6 -> 12.0 mm
- net ENABLE: track 25.0 -> 23.6 mm
- added copper zone on layer 1, net VBUS
Changed lines of the file:
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@@
 <setting verticaltext="up"/>
 </settings>
-<grid distance="25" unitdist="mil" unit="mil" style="lines" multiple="1" display="yes" altdistance="5" altunitdist="mil" altunit="mil"/>
+<grid distance="1" unitdist="mil" unit="mil" style="lines" multiple="1" display="yes" altdistance="5" altunitdist="mil" altunit="mil"/>
 <layers>
 <layer number="1" name="Top" color="4" fill="1" visible="yes" active="yes"/>
@@
 </class>
 </classes>
-<designrules name="default">
-<description language="de">&lt;b&gt;EAGLE Design Rules&lt;/b&gt;
+<designrules name="OshPark">
+<description language="en">&lt;b&gt;OSH Park Design Rules&lt;/b&gt;
 &lt;p&gt;
-Die Standard-Design-Rules sind so gewählt, dass sie für
-die meisten Anwendungen passen. Sollte ihre Platine
-besondere Anforderungen haben, treffen Sie die erforderlichen
-Einstellungen hier und speichern die Design Rules unter
-einem neuen Namen ab.</description>
-<description language="en">&lt;b&gt;EAGLE Design Rules&lt;/b&gt;
+Please make sure your boards conform to these design rules.
+&lt;/p&gt;
 &lt;p&gt;
-The default Design Rules have been set to cover
-a wide range of applications. Your particular design
-may have different requirements, so please make the
-necessary adjustments and save your customized
-design rules under a new name.</description>
+Note, that not all DRC settings must be set by the manufacturer. Several can be adjusted for the design, including those listed on our docs page here.
+&lt;a href=&quot;http://docs.oshpark.com/design-tools/eagle/design-rules-files/&quot;&gt;Adjustable Settings&lt;/a&gt;
+&lt;/p&gt;</description>
 <param name="layerSetup" value="(1*16)"/>
-<param name="mtCopper" value="0.035mm 0.035mm 0.035mm 0.035mm 0.035mm 0.035mm 0.035mm 0.035mm 0.035mm 0.035mm 0.035mm 0.035mm 0.035mm 0.035mm 0.035mm 0.035mm"/>
-<param name="mtIsolate" value="1.5mm 0.15mm 0.2mm 0.15mm 0.2mm 0.15mm 0.2mm 0.15mm 0.2mm 0.15mm 0.2mm 0.15mm 0.2mm 0.15mm 0.2mm"/>
+<param name="mtCopper" value="0.035559375mm 0.0356mm 0.0356mm 0.0356mm 0.0356mm 0.0356mm 0.0356mm 0.0356mm 0.0356mm 0.0356mm 0.0356mm 0.0356mm 0.0356mm 0.0356mm 0.0356mm 0.035559375mm"/>
+<param name="mtIsolate" value="1.6mm 0.1499mm 0.2007mm 0.1499mm 0.2007mm 0.1499mm 0.2007mm 0.1499mm 0.2007mm 0.1499mm 0.2007mm 0.1499mm 0.2007mm 0.1499mm 0.2007mm"/>
 <param name="mdWireWire" value="6mil"/>
 <param name="mdWirePad" value="6mil"/>
@@
 <param name="mdSmdVia" value="6mil"/>
 <param name="mdSmdSmd" value="6mil"/>
-<param name="mdViaViaSameLayer" value="6mil"/>
+<param name="mdViaViaSameLayer" value="8mil"/>
 <param name="mnLayersViaInSmd" value="2"/>
-<param name="mdCopperDimension" value="40mil"/>
+<param name="mdCopperDimension" value="15mil"/>
 <param name="mdDrill" value="6mil"/>
 <param name="mdSmdStop" value="0mil"/>
 <param name="msWidth" value="6mil"/>
-<param name="msDrill" value="0.35mm"/>
-<param name="msMicroVia" value="9.99mm"/>
+<param name="msDrill" value="10mil"/>
+<param name="msMicroVia" value="10mil"/>
 <param name="msBlindViaRatio" value="0.5"/>
 <param name="rvPadTop" value="0.25"/>
@@
 <param name="rvMicroViaOuter" value="0.25"/>
 <param name="rvMicroViaInner" value="0.25"/>
-<param name="rlMinPadTop" value="10mil"/>
+<param name="rlMinPadTop" value="5mil"/>
 <param name="rlMaxPadTop" value="20mil"/>
-<param name="rlMinPadInner" value="10mil"/>
+<param name="rlMinPadInner" value="5mil"/>
 <param name="rlMaxPadInner" value="20mil"/>
-<param name="rlMinPadBottom" value="10mil"/>
+<param name="rlMinPadBottom" value="5mil"/>
 <param name="rlMaxPadBottom" value="20mil"/>
-<param name="rlMinViaOuter" value="8mil"/>
+<param name="rlMinViaOuter" value="5mil"/>
 <param name="rlMaxViaOuter" value="20mil"/>
-<param name="rlMinViaInner" value="8mil"/>
+<param name="rlMinViaInner" value="5mil"/>
 <param name="rlMaxViaInner" value="20mil"/>
-<param name="rlMinMicroViaOuter" value="4mil"/>
+<param name="rlMinMicroViaOuter" value="5mil"/>
 <param name="rlMaxMicroViaOuter" value="20mil"/>
-<param name="rlMinMicroViaInner" value="4mil"/>
+<param name="rlMinMicroViaInner" value="5mil"/>
 <param name="rlMaxMicroViaInner" value="20mil"/>
 <param name="psTop" value="-1"/>
@@
 <param name="mvStopFrame" value="1"/>
 <param name="mvCreamFrame" value="0"/>
-<param name="mlMinStopFrame" value="4mil"/>
-<param name="mlMaxStopFrame" value="4mil"/>
+<param name="mlMinStopFrame" value="2.5mil"/>
+<param name="mlMaxStopFrame" value="2.5mil"/>
 <param name="mlMinCreamFrame" value="0mil"/>
 <param name="mlMaxCreamFrame" value="0mil"/>
@@
 <wire x1="16.315" y1="9.723" x2="16.94" y2="9.723" width="0.3048" layer="1"/>
 <wire x1="16.94" y1="9.723" x2="17.515" y2="10.298" width="0.3048" layer="1"/>
-<wire x1="10.398" y1="9.287" x2="10.398" y2="9.414" width="0.3048" layer="1"/>
-<wire x1="10.398" y1="9.287" x2="9.398" y2="10.287" width="0.3048" layer="1"/>
-<wire x1="11.363" y1="9.414" x2="10.398" y2="9.414" width="0.3048" layer="1"/>
-<wire x1="18.09" y1="9.723" x2="18.415" y2="9.398" width="0.3048" layer="1"/>
-<wire x1="18.74" y1="9.723" x2="18.415" y2="9.398" width="0.3048" layer="1"/>
-<wire x1="19.39" y1="10.373" x2="19.315" y2="10.298" width="0.3048" layer="1"/>
-<wire x1="18.74" y1="12.695" x2="18.481" y2="12.954" width="0.3048" layer="1"/>
-<wire x1="18.09" y1="12.563" x2="18.481" y2="12.954" width="0.3048" layer="1"/>
-<wire x1="18.796" y1="12.954" x2="18.481" y2="12.954" width="0.3048" layer="1"/>
 <wire x1="18.415" y1="9.398" x2="17.44" y2="8.423" width="0.3048" layer="1"/>
 <wire x1="17.44" y1="8.423" x2="17.44" y2="7.298" width="0.3048" layer="1"/>
 <via x="4.318" y="5.715" extent="1-16" drill="0.35"/>
 <via x="9.398" y="10.287" extent="1-16" drill="0.35"/>
-<wire x1="10.398" y1="8.449" x2="10.398" y2="9.287" width="0.3048" layer="1"/>
 <wire x1="9.398" y1="10.414" x2="9.398" y2="10.287" width="0.2032" layer="1"/>
 <via x="10.795" y="15.24" extent="1-16" drill="0.35"/>
@@
 <via x="26.4414" y="7.5438" extent="1-16" drill="0.35"/>
 <via x="26.416" y="8.763" extent="1-16" drill="0.35"/>
-<wire x1="10.398" y1="8.449" x2="10.16" y2="5.969" width="0" layer="19" extent="1-1"/>
 <via x="5.2832" y="5.715" extent="1-16" drill="0.35"/>
+<via x="11.0744" y="8.7122" extent="1-16" drill="0.35"/>
 </signal>
 <signal name="N$1">
@@
 <contactref element="U1" pad="4"/>
 <contactref element="L1" pad="P$2"/>
-<wire x1="21.844" y1="10.373" x2="23.403" y2="10.373" width="0.3048" layer="1"/>
-<wire x1="23.403" y1="10.373" x2="24.003" y2="10.973" width="0.3048" layer="1"/>
 <polygon width="0.1016" layer="1" thermals="no">
 <vertex x="20.0406" y="10.4902"/>
@@
 <contactref element="C6" pad="1"/>
 <contactref element="J2" pad="2"/>
-<wire x1="21.927" y1="8.423" x2="22.222" y2="8.128" width="0.3048" layer="1"/>
-<wire x1="22.222" y1="7.49" x2="22.222" y2="7.874" width="0.3048" layer="1"/>
-<wire x1="22.222" y1="7.874" x2="22.222" y2="8.128" width="0.3048" layer="1"/>
-<wire x1="22.03" y1="7.298" x2="22.222" y2="7.49" width="0.3048" layer="1"/>
-<wire x1="22.037" y1="7.689" x2="22.222" y2="7.874" width="0.3048" layer="1"/>
 <via x="23.622" y="8.128" extent="1-16" drill="0.35"/>
 <wire x1="22.225" y1="16.51" x2="25.6032" y2="13.1318" width="0.8128" layer="16"/>
@@
 <via x="5.2832" y="14.5288" extent="1-16" drill="0.35"/>
 <wire x1="5.2832" y1="14.5288" x2="4.3332" y2="14.5288" width="0.3048" layer="1"/>
-<via x="13.462" y="10.16" extent="1-16" drill="0.35"/>
+<via x="13.8176" y="8.9154" extent="1-16" drill="0.35"/>
 <wire x1="5.2832" y1="14.5288" x2="5.2832" y2="8.0518" width="0.3048" layer="16"/>
 <wire x1="6.6294" y1="6.7056" x2="10.1092" y2="6.7056" width="0.3048" layer="16"/>
-<wire x1="10.1092" y1="6.7056" x2="13.462" y2="10.0584" width="0.3048" layer="16"/>
-<wire x1="13.462" y1="10.0584" x2="13.462" y2="10.16" width="0.3048" layer="16"/>
+<wire x1="10.1092" y1="6.7056" x2="12.319" y2="8.9154" width="0.3048" layer="16"/>
+<wire x1="13.8176" y1="8.9154" x2="12.319" y2="8.9154" width="0.3048" layer="16"/>
 <wire x1="5.2832" y1="8.0518" x2="6.6294" y2="6.7056" width="0.3048" layer="16"/>
-<wire x1="13.462" y1="10.16" x2="13.716" y2="9.906" width="0.3048" layer="1"/>
-<wire x1="13.716" y1="9.906" x2="13.716" y2="9.271" width="0.3048" layer="1"/>
-<wire x1="13.716" y1="9.271" x2="14.097" y2="8.89" width="0.3048" layer="1"/>
 <wire x1="15.70705" y1="9.073" x2="16.315" y2="9.073" width="0.3048" layer="1"/>
-<wire x1="14.097" y1="8.89" x2="15.52405" y2="8.89" width="0.3048" layer="1"/>
 <wire x1="15.52405" y1="8.89" x2="15.70705" y2="9.073" width="0.3048" layer="1"/>
 <wire x1="4.3332" y1="14.859" x2="4.3332" y2="14.5288" width="0.3048" layer="1"/>
+<wire x1="15.52405" y1="8.89" x2="13.843" y2="8.89" width="0.3048" layer="1"/>
+<wire x1="13.843" y1="8.89" x2="13.8176" y2="8.9154" width="0.3048" layer="1"/>
 </signal>
 <signal name="N$5">
@@
 <wire x1="6.985" y1="16.51" x2="9.398" y2="14.097" width="0.8128" layer="1"/>
 <wire x1="9.398" y1="14.097" x2="9.398" y2="13.335" width="0.8128" layer="1"/>
+<polygon width="0.1524" layer="1" thermals="no">
+<vertex x="8.8392" y="12.0904"/>
+<vertex x="9.9568" y="12.0904"/>
+<vertex x="9.9568" y="13.0556"/>
+<vertex x="9.398" y="13.6144"/>
+<vertex x="8.8392" y="13.0556"/>
+</polygon>
 </signal>
 <signal name="VLIPO">
